Commit message: Add colors to Gazebo simulation

File: urdf/spotmicroai.urdf.xacro (robot description, xacro)
@@ -58,4 +58,7 @@
       </inertial>
     </link>
+    <gazebo reference="${name}">
+      <material>Gazebo/FlatBlack</material>
+    </gazebo>
   </xacro:macro>
   <xacro:macro name="gen_shoulder_joint" params="pos shiftx shifty">
@@ -87,4 +90,7 @@
       </visual>
     </link>
+    <gazebo reference="${name}_cover">
+      <material>Gazebo/ZincYellow</material>
+    </gazebo>
     <link name="${name}">
       <visual>
@@ -102,9 +108,4 @@
         </xacro:unless>
         <material name="black"/>
-<!--        <geometry>
-          <box size="0.028 0.036 ${leg_length}"/>
-        </geometry>
-        <origin rpy="0.0 0.0 0.0" xyz="0.0 0.0 -0.050"/>
-        <material name="yellow"/>-->
       </visual>
       <collision>
@@ -119,4 +120,7 @@
       </inertial>
     </link>
+    <gazebo reference="${name}">
+      <material>Gazebo/FlatBlack</material>
+    </gazebo>
   </xacro:macro>
   <xacro:macro name="gen_leg_joint" params="pos shift">
@@ -130,8 +134,8 @@
     </joint>
     <joint name="${pos}_leg_cover_joint" type="fixed">
-    <parent link="${pos}_leg_link"/>
-    <child link="${pos}_leg_link_cover"/>
-        <origin xyz="0 0 0"/>
-  </joint>
+      <parent link="${pos}_leg_link"/>
+      <child link="${pos}_leg_link_cover"/>
+      <origin xyz="0 0 0"/>
+    </joint>
   </xacro:macro>
   <xacro:macro name="gen_foot" params="name left">
@@ -163,4 +167,7 @@
       </inertial>
     </link>
+    <gazebo reference="${name}">
+      <material>Gazebo/FlatBlack</material>
+    </gazebo>
   </xacro:macro>
   <xacro:macro name="gen_foot_joint" params="pos">
@@ -195,4 +202,7 @@
       </inertial>
     </link>
+    <gazebo reference="${name}">
+      <material>Gazebo/Grey</material>
+    </gazebo>
   </xacro:macro>
  <xacro:macro name="gen_toe_joint" params="pos">
@@ -233,4 +243,7 @@
     </inertial>
   </link>
+  <gazebo reference="base_link">
+    <material>Gazebo/FlatBlack</material>
+  </gazebo>
   <!-- Lidar Backpack -->
    <link name="lidar_link">
@@ -253,4 +266,7 @@
     </inertial>
   </link>
+  <gazebo reference="lidar_link">
+    <material>Gazebo/FlatBlack</material>
+  </gazebo>
   <joint name="base_lidar" type="fixed">
     <parent link="base_link"/>
@@ -277,4 +293,7 @@
     </inertial>
   </link>
+  <gazebo reference="rear_link">
+    <material>Gazebo/ZincYellow</material>
+  </gazebo>
   <joint name="base_rear" type="fixed">
     <parent link="base_link"/>
@@ -300,4 +319,7 @@
     </inertial>
   </link>
+  <gazebo reference="front_link">
+    <material>Gazebo/ZincYellow</material>
+  </gazebo>
   <joint name="base_front" type="fixed">
     <parent link="base_link"/>
