Commit message: fixed orientation

File: urdf/spotmicroai.urdf (robot description, URDF)
Before this commit: robot SpotMicroAI, 24 links, 23 joints
Links:
- removed link lidar_link
- added link base_inertia, mass 2.80; collision box size=0.14 0.11 0.07; visual mesh filename=package://spotmicro_description/meshes/stl/mainbody.stl scale=0.001 0.001 0.001
- link base_link: mass 2.80 -> None; geometry 
- link front_left_foot_link: geometry collision box size=0.026 0.020 0.13; visual mesh filename=package://spotmicro_description/meshes/stl/lfoot.stl scale=0.001 0.001 0.001
- link front_left_leg_link: geometry collision box size=0.028 0.036 0.109; visual mesh filename=package://spotmicro_description/meshes/stl/larm.stl scale=0.001 0.001 0.001
- link front_right_foot_link: geometry collision box size=0.026 0.020 0.13; visual mesh filename=package://spotmicro_description/meshes/stl/rfoot.stl scale=0.001 0.001 0.001
- link front_right_leg_link: geometry collision box size=0.028 0.036 0.109; visual mesh filename=package://spotmicro_description/meshes/stl/rarm.stl scale=0.001 0.001 0.001
- link rear_left_foot_link: geometry collision box size=0.026 0.020 0.13; visual mesh filename=package://spotmicro_description/meshes/stl/lfoot.stl scale=0.001 0.001 0.001
- link rear_left_leg_link: geometry collision box size=0.028 0.036 0.109; visual mesh filename=package://spotmicro_description/meshes/stl/larm.stl scale=0.001 0.001 0.001
- link rear_right_foot_link: geometry collision box size=0.026 0.020 0.13; visual mesh filename=package://spotmicro_description/meshes/stl/rfoot.stl scale=0.001 0.001 0.001
- link rear_right_leg_link: geometry collision box size=0.028 0.036 0.109; visual mesh filename=package://spotmicro_description/meshes/stl/rarm.stl scale=0.001 0.001 0.001
Joints:
- removed joint base_lidar
- added joint base_inertia_joint: type fixed, parent base_link, child base_inertia
- joint front_left_foot: origin xyz=-0.01 0 -0.12 rpy=0 0 0 -> xyz=0.014 0 -0.109 rpy=0 0 0
- joint front_left_leg: origin xyz=0 -0.052 0 rpy=0 0 0 -> xyz=0 0.055 0 rpy=0 0 0
- joint front_left_shoulder: origin xyz=-0.093 -0.036 0 rpy=0 0 0 -> xyz=0.093 0.0395 0 rpy=0 0 0
- joint front_left_toe: origin xyz=0 0 -0.115 -> xyz=0 0 -0.13
- joint front_right_foot: origin xyz=-0.01 0 -0.12 rpy=0 0 0 -> xyz=0.014 0 -0.109 rpy=0 0 0
- joint front_right_leg: origin xyz=0 0.052 0 rpy=0 0 0 -> xyz=0 -0.055 0 rpy=0 0 0
- joint front_right_shoulder: origin xyz=-0.093 0.036 0 rpy=0 0 0 -> xyz=0.093 -0.0395 0 rpy=0 0 0
- joint front_right_toe: origin xyz=0 0 -0.115 -> xyz=0 0 -0.13
- joint rear_left_foot: origin xyz=-0.01 0 -0.12 rpy=0 0 0 -> xyz=0.014 0 -0.109 rpy=0 0 0
- joint rear_left_leg: origin xyz=0 -0.052 0 rpy=0 0 0 -> xyz=0 0.055 0 rpy=0 0 0
- joint rear_left_shoulder: origin xyz=0.093 -0.036 0 rpy=0 0 0 -> xyz=-0.093 0.0395 0 rpy=0 0 0
- joint rear_left_toe: origin xyz=0 0 -0.115 -> xyz=0 0 -0.13
- joint rear_right_foot: origin xyz=-0.01 0 -0.12 rpy=0 0 0 -> xyz=0.014 0 -0.109 rpy=0 0 0
- joint rear_right_leg: origin xyz=0 0.052 0 rpy=0 0 0 -> xyz=0 -0.055 0 rpy=0 0 0
- joint rear_right_shoulder: origin xyz=0.093 0.036 0 rpy=0 0 0 -> xyz=-0.093 -0.0395 0 rpy=0 0 0
- joint rear_right_toe: origin xyz=0 0 -0.115 -> xyz=0 0 -0.13

File: urdf/spotmicroai.urdf.xacro (robot description, xacro)
@@ -1,333 +1,295 @@
-<?xml version="1.0"?>
+<?xml version="1.0" encoding="UTF-8"?>
 <robot xmlns:xacro="http://www.ros.org/wiki/xacro" name="SpotMicroAI">
-  <material name="yellow">
-    <color rgba="0.92 0.83 0.0 1"/>
-  </material>
-  <material name="black">
-    <color rgba="0.1 0.1 0.1 1"/>
-  </material>
-  <material name="grey">
-    <color rgba="0.6 0.6 0.6 1"/>
-  </material>
-  <!-- Params -->
-  <xacro:property name="body_length" value="0.140" />
-  <xacro:property name="body_width" value="0.110" />
-  <xacro:property name="body_height" value="0.070" />
-  <xacro:property name="lidar_length" value="0.0985" />
-  <xacro:property name="lidar_width" value="0.0577" />
-  <xacro:property name="lidar_height" value="0.070" />
-  <xacro:property name="front_length" value="0.058" />
-  <xacro:property name="rear_length" value="0.040" />
-  <xacro:property name="shoulder_length" value="0.044" />
-  <xacro:property name="shoulder_width" value="0.038" />
-  <xacro:property name="leg_length" value="0.120" />
-  <xacro:property name="foot_length" value="0.115" />
-  <xacro:property name="toe_radius" value="0.020" />
-  <!--  <xacro:property name="toe_radius" value="0.014" /> -->
-  <xacro:property name="toe_width" value="0.020" />
-  <xacro:property name="shift" value="0.052" />
-  <xacro:property name="shiftx" value="0.093" />
-  <xacro:property name="shifty" value="0.036" />
-  <!-- Macros -->
-  <xacro:macro name="gen_shoulder" params="name left">
-    <link name="${name}">
+   <material name="yellow">
+      <color rgba="0.92 0.83 0.0 1" />
+   </material>
+   <material name="black">
+      <color rgba="0.1 0.1 0.1 1" />
+   </material>
+   <material name="grey">
+      <color rgba="0.6 0.6 0.6 1" />
+   </material>
+   <!-- Params -->
+   <xacro:property name="body_length" value="0.140" />
+   <xacro:property name="body_width" value="0.110" />
+   <xacro:property name="body_height" value="0.070" />
+   <xacro:property name="lidar_length" value="0.0985" />
+   <xacro:property name="lidar_width" value="0.0577" />
+   <xacro:property name="lidar_height" value="0.070" />
+   <xacro:property name="front_length" value="0.058" />
+   <xacro:property name="rear_length" value="0.040" />
+   <xacro:property name="shoulder_length" value="0.044" />
+   <xacro:property name="shoulder_width" value="0.038" />
+   <xacro:property name="leg_length" value="0.109" />
+   <xacro:property name="foot_length" value="0.13" />
+   <xacro:property name="toe_radius" value="0.020" />
+   <!--  <xacro:property name="toe_radius" value="0.014" /> -->
+   <xacro:property name="toe_width" value="0.020" />
+   <xacro:property name="shift" value="0.055" />
+   <xacro:property name="shiftx" value="0.093" />
+   <xacro:property name="shifty" value="0.0395" />
+   <!-- Macros -->
+   <xacro:macro name="gen_shoulder" params="name left">
+      <link name="${name}">
+         <visual>
+            <xacro:if value="${left}">
+               <geometry>
+                  <mesh filename="package://spotmicro_description/meshes/stl/lshoulder.stl" scale="0.001 0.001 0.001" />
+               </geometry>
+               <origin rpy="0 0 3.1416" xyz="0.135 0.0163 -0.0195" />
+            </xacro:if>
+            <xacro:unless value="${left}">
+               <geometry>
+                  <mesh filename="package://spotmicro_description/meshes/stl/rshoulder.stl" scale="0.001 0.001 0.001" />
+               </geometry>
+               <origin rpy="0 0 3.1416" xyz="0.135 0.0938 -0.0205" />
+            </xacro:unless>
+            <material name="black" />
+         </visual>
+         <collision>
+            <geometry>
+               <box size="${shoulder_length} ${shoulder_width} ${body_height}" />
+            </geometry>
+            <origin rpy="0 0 0" xyz="0 0 0" />
+         </collision>
+         <inertial>
+            <mass value="0.10" />
+            <inertia ixx="100" ixy="0" ixz="0" iyy="100" iyz="0" izz="100" />
+         </inertial>
+      </link>
+   </xacro:macro>
+   <xacro:macro name="gen_shoulder_joint" params="pos shiftx shifty">
+      <joint name="${pos}_shoulder" type="revolute">
+         <parent link="base_link" />
+         <child link="${pos}_shoulder_link" />
+         <axis xyz="1 0 0" />
+         <origin rpy="0 0 0" xyz="${shiftx} ${shifty} 0" />
+         <limit effort="1000.0" lower="-0.548" upper="0.548" velocity="0.7" />
+         <dynamics damping="0.0" friction="0.5" />
+      </joint>
+   </xacro:macro>
+   <xacro:macro name="gen_leg" params="name left">
+      <link name="${name}_cover">
+         <visual>
+            <xacro:if value="${left}">
+               <geometry>
+                  <mesh filename="package://spotmicro_description/meshes/stl/larm_cover.stl" scale="0.001 0.001 0.001" />
+               </geometry>
+               <origin rpy="0 0 3.1416" xyz="0.134 -0.04 -0.0095" />
+            </xacro:if>
+            <xacro:unless value="${left}">
+               <geometry>
+                  <mesh filename="package://spotmicro_description/meshes/stl/rarm_cover.stl" scale="0.001 0.001 0.001" />
+               </geometry>
+               <origin rpy="0 0 3.1416" xyz="0.134 0.149 -0.0095" />
+            </xacro:unless>
+            <material name="yellow" />
+         </visual>
+      </link>
+      <link name="${name}">
+         <visual>
+            <xacro:if value="${left}">
+               <geometry>
+                  <mesh filename="package://spotmicro_description/meshes/stl/larm.stl" scale="0.001 0.001 0.001" />
+               </geometry>
+               <origin rpy="0 0 3.1416" xyz="0.134 -0.04 -0.0095" />
+            </xacro:if>
+            <xacro:unless value="${left}">
+               <geometry>
+                  <mesh filename="package://spotmicro_description/meshes/stl/rarm.stl" scale="0.001 0.001 0.001" />
+               </geometry>
+               <origin rpy="0 0 3.1416" xyz="0.134 0.149 -0.0095" />
+            </xacro:unless>
+            <material name="black" />
+         </visual>
+         <collision>
+            <origin rpy="0.0 0.0 0.0" xyz="0.0 0.0 -0.050" />
+            <geometry>
+               <box size="0.028 0.036 ${leg_length}" />
+            </geometry>
+         </collision>
+         <inertial>
+            <mass value="0.15" />
+            <inertia ixx="1000" ixy="0" ixz="0" iyy="1000" iyz="0" izz="1000" />
+         </inertial>
+      </link>
+      <gazebo reference="${name}_cover">
+         <material>Gazebo/ZincYellow</material>
+      </gazebo>
+   </xacro:macro>
+   <xacro:macro name="gen_leg_joint" params="pos shift">
+      <joint name="${pos}_leg" type="revolute">
+         <parent link="${pos}_shoulder_link" />
+         <child link="${pos}_leg_link" />
+         <axis xyz="0 1 0" />
+         <origin rpy="0 0 0" xyz="0 ${shift} 0" />
+         <limit effort="1000.0" lower="-2.666" upper="1.548" velocity="0.5" />
+         <dynamics damping="0.0" friction="0.0" />
+      </joint>
+      <joint name="${pos}_leg_cover_joint" type="fixed">
+         <parent link="${pos}_leg_link" />
+         <child link="${pos}_leg_link_cover" />
+         <origin xyz="0 0 0" />
+      </joint>
+   </xacro:macro>
+   <xacro:macro name="gen_foot" params="name left">
+      <link name="${name}">
+         <visual>
+            <xacro:if value="${left}">
+               <geometry>
+                  <mesh filename="package://spotmicro_description/meshes/stl/lfoot.stl" scale="0.001 0.001 0.001" />
+               </geometry>
+               <origin rpy="0 0 3.1416 " xyz="0.1195 -0.04 0.099" />
+            </xacro:if>
+            <xacro:unless value="${left}">
+               <geometry>
+                  <mesh filename="package://spotmicro_description/meshes/stl/rfoot.stl" scale="0.001 0.001 0.001" />
+               </geometry>
+               <origin rpy="0 0 3.1416" xyz="0.1195 0.149 0.099" />
+            </xacro:unless>
+            <material name="black" />
+         </visual>
+         <collision>
+            <geometry>
+               <box size="0.026 0.020 ${foot_length}" />
+            </geometry>
+            <origin rpy="0.0 0.0 0.0" xyz="0.0 0.0 -0.050" />
+         </collision>
+         <inertial>
+            <mass value="0.1" />
+            <inertia ixx="1000" ixy="0" ixz="0" iyy="1000" iyz="0" izz="1000" />
+         </inertial>
+      </link>
+   </xacro:macro>
+   <xacro:macro name="gen_foot_joint" params="pos">
+      <joint name="${pos}_foot" type="revolute">
+         <parent link="${pos}_leg_link" />
+         <child link="${pos}_foot_link" />
+         <axis xyz="0 1 0" />
+         <origin rpy="0 0 0" xyz="0.014 0 -${leg_length}" />
+         <limit effort="1000.0" lower="-0.1" upper="2.59" velocity="0.5" />
+         <dynamics damping="0.0" friction="0.5" />
+      </joint>
+   </xacro:macro>
+   <xacro:macro name="gen_toe" params="name">
+      <link name="${name}">
+         <visual>
+            <geometry>
+               <mesh filename="package://spotmicro_description/meshes/stl/foot.stl" scale="0.001 0.001 0.001" />
+            </geometry>
+            <origin rpy="0 0.40010 0" xyz="0 -0.01 0.015" />
+            <material name="grey" />
+         </visual>
+         <collision>
+            <geometry>
+               <sphere radius="${toe_radius}" />
+            </geometry>
+            <origin rpy="0 0 0" xyz="0 0 0" />
+            <contact_coefficients mu="1.1" />
+         </collision>
+         <inertial>
+            <mass value="0.05" />
+            <inertia ixx="1000" ixy="0" ixz="0" iyy="1000" iyz="0" izz="1000" />
+         </inertial>
+      </link>
+   </xacro:macro>
+   <xacro:macro name="gen_toe_joint" params="pos">
+      <joint name="${pos}_toe" type="fixed">
+         <parent link="${pos}_foot_link" />
+         <child link="${pos}_toe_link" />
+         <origin xyz="0 0 -${foot_length}" />
+      </joint>
+   </xacro:macro>
+   <xacro:macro name="gen_full_leg_joint" params="pos shiftx shifty shift left">
+      <xacro:gen_shoulder name="${pos}_shoulder_link" left="${left}" />
+      <xacro:gen_leg name="${pos}_leg_link" left="${left}" />
+      <xacro:gen_foot name="${pos}_foot_link" left="${left}" />
+      <xacro:gen_toe name="${pos}_toe_link" />
+      <xacro:gen_shoulder_joint pos="${pos}" shiftx="${shiftx}" shifty="${shifty}" />
+      <xacro:gen_leg_joint pos="${pos}" shift="${shift}" />
+      <xacro:gen_foot_joint pos="${pos}" />
+      <xacro:gen_toe_joint pos="${pos}" />
+   </xacro:macro>
+   <!-- Robot Body -->
+   <link name="base_link"/>
+   <link name="base_inertia">
       <visual>
-        <xacro:if value="${left}">
-        <geometry>
-          <mesh filename="package://spotmicro_description/meshes/stl/lshoulder.stl" scale="0.001 0.001 0.001"/>
-        </geometry>
-        <origin rpy="0 0 0" xyz="-0.135 -0.02 -0.01"/>
-        </xacro:if>
-        <xacro:unless value="${left}">
-        <geometry>
-          <mesh filename="package://spotmicro_description/meshes/stl/rshoulder.stl" scale="0.001 0.001 0.001"/>
-        </geometry>
-        <origin rpy="0 0 0" xyz="-0.135 -0.09 -0.01"/>
-        </xacro:unless>
-        <material name="black"/>
+         <geometry>
+            <mesh filename="package://spotmicro_description/meshes/stl/mainbody.stl" scale="0.001 0.001 0.001" />
+         </geometry>
+         <material name="black" />
+         <origin rpy="0 0 3.1416" xyz="0.0425 0.055 -0.02" />
       </visual>
       <collision>
-        <geometry>
-          <box size="${shoulder_length} ${shoulder_width} ${body_height}"/>
-        </geometry>
-        <origin rpy="0 0 0" xyz="0 0 0"/>
+         <geometry>
+            <box size="${body_length} ${body_width} ${body_height}" />
+         </geometry>
+         <origin rpy="0 0 3.1416" xyz="0 0 0" />
       </collision>
       <inertial>
-        <mass value="0.10"/>
-        <inertia ixx="100" ixy="0" ixz="0" iyy="100" iyz="0" izz="100" />
+         <mass value="2.80" />
+         <inertia ixx="100" ixy="0" ixz="0" iyy="100" iyz="0" izz="100" />
       </inertial>
-    </link>
-    <gazebo reference="${name}">
-      <material>Gazebo/FlatBlack</material>
-    </gazebo>
-  </xacro:macro>
-  <xacro:macro name="gen_shoulder_joint" params="pos shiftx shifty">
-    <joint name="${pos}_shoulder" type="revolute">
-      <parent link="base_link"/>
-      <child link="${pos}_shoulder_link"/>
-      <axis xyz="1 0 0"/>
-      <origin rpy="0 0 0" xyz="${shiftx} ${shifty} 0"/>
-      <limit effort="1000.0" lower="-0.548" upper="0.548" velocity="0.7"/>
-      <dynamics damping="0.0" friction="0.5"/>
-    </joint>
-  </xacro:macro>
-  <xacro:macro name="gen_leg" params="name left">
-    <link name="${name}_cover">
+   </link>
+   <joint name="base_inertia_joint" type="fixed">
+      <parent link="base_link" />
+      <child link="base_inertia" />
+   </joint>
+   <link name="rear_link">
       <visual>
-        <xacro:if value="${left}">
-        <geometry>
-          <mesh filename="package://spotmicro_description/meshes/stl/larm_cover.stl" scale="0.001 0.001 0.001"/>
-        </geometry>
-        <origin rpy="0 0 0" xyz="-0.125 0.04 -0.02"/>
-        </xacro:if>
-        <xacro:unless value="${left}">
-        <geometry>
-          <mesh filename="package://spotmicro_description/meshes/stl/rarm_cover.stl" scale="0.001 0.001 0.001"/>
-        </geometry>
-        <origin rpy="0 0 0" xyz="-0.125 -0.15 -0.02"/>
-        </xacro:unless>
-        <material name="yellow"/>
-      </visual>
-    </link>
-    <gazebo reference="${name}_cover">
-      <material>Gazebo/ZincYellow</material>
-    </gazebo>
-    <link name="${name}">
-      <visual>
-        <xacro:if value="${left}">
-        <geometry>
-          <mesh filename="package://spotmicro_description/meshes/stl/larm.stl" scale="0.001 0.001 0.001"/>
-        </geometry>
-        <origin rpy="0 0 0" xyz="-0.125 0.04 -0.02"/>
-        </xacro:if>
-        <xacro:unless value="${left}">
-        <geometry>
-          <mesh filename="package://spotmicro_description/meshes/stl/rarm.stl" scale="0.001 0.001 0.001"/>
-        </geometry>
-        <origin rpy="0 0 0" xyz="-0.125 -0.15 -0.02"/>
-        </xacro:unless>
-        <material name="black"/>
+         <geometry>
+            <mesh filename="package://spotmicro_description/meshes/stl/backpart.stl" scale="0.001 0.001 0.001" />
+         </geometry>
+         <origin rpy="0 0 3.1416" xyz="0.042 0.055 -0.0195" />
+         <material name="yellow" />
       </visual>
       <collision>
-        <origin rpy="0.0 0.0 0.0" xyz="0.0 0.0 -0.050"/>
-        <geometry>
-          <box size="0.028 0.036 ${leg_length}"/>
-        </geometry>
+         <geometry>
+            <box size="${rear_length} ${body_width} ${body_height}" />
+         </geometry>
+         <origin rpy="0 0 0" xyz="-0.135 0 0" />
       </collision>
       <inertial>
-        <mass value="0.15"/>
-        <inertia ixx="1000" ixy="0" ixz="0" iyy="1000" iyz="0" izz="1000" />
+         <mass value="0.20" />
+         <inertia ixx="100" ixy="0" ixz="0" iyy="100" iyz="0" izz="100" />
       </inertial>
-    </link>
-    <gazebo reference="${name}">
-      <material>Gazebo/FlatBlack</material>
-    </gazebo>
-  </xacro:macro>
-  <xacro:macro name="gen_leg_joint" params="pos shift">
-    <joint name="${pos}_leg" type="revolute">
-      <parent link="${pos}_shoulder_link"/>
-      <child link="${pos}_leg_link"/>
-      <axis xyz="0 1 0"/>
-      <origin rpy="0 0 0" xyz="0 ${shift} 0"/>
-      <limit effort="1000.0" lower="-2.666" upper="1.548" velocity="0.5"/>
-      <dynamics damping="0.0" friction="0.0"/>
-    </joint>
-    <joint name="${pos}_leg_cover_joint" type="fixed">
-      <parent link="${pos}_leg_link"/>
-      <child link="${pos}_leg_link_cover"/>
-      <origin xyz="0 0 0"/>
-    </joint>
-  </xacro:macro>
-  <xacro:macro name="gen_foot" params="name left">
-    <link name="${name}">
+   </link>
+   <joint name="base_rear" type="fixed">
+      <parent link="base_link" />
+      <child link="rear_link" />
+   </joint>
+   <gazebo reference="rear_link">
+      <material>Gazebo/ZincYellow</material>
+   </gazebo>
+   <link name="front_link">
       <visual>
-        <xacro:if value="${left}">
-        <geometry>
-          <mesh filename="package://spotmicro_description/meshes/stl/lfoot.stl" scale="0.001 0.001 0.001"/>
-        </geometry>
-        <origin rpy="0 0 0" xyz="-0.120 0.04 0.1"/>
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