Commit message: Add transmission and change joint limits

File: urdf/spotmicroai.urdf (robot description, URDF)
Before this commit: robot SpotMicroAI, 24 links, 23 joints
Joints:
- joint front_left_foot: limit lower=-0.1 upper=2.59 effort=1000.0 velocity=0.5 -> lower=-2.59 upper=0.1 effort=1000.0 velocity=0.5
- joint front_right_foot: limit lower=-0.1 upper=2.59 effort=1000.0 velocity=0.5 -> lower=-2.59 upper=0.1 effort=1000.0 velocity=0.5
- joint rear_left_foot: limit lower=-0.1 upper=2.59 effort=1000.0 velocity=0.5 -> lower=-2.59 upper=0.1 effort=1000.0 velocity=0.5
- joint rear_right_foot: limit lower=-0.1 upper=2.59 effort=1000.0 velocity=0.5 -> lower=-2.59 upper=0.1 effort=1000.0 velocity=0.5

File: urdf/spotmicroai.urdf.xacro (robot description, xacro)
@@ -65,7 +65,17 @@
          <axis xyz="1 0 0" />
          <origin rpy="0 0 0" xyz="${shiftx} ${shifty} 0" />
-         <limit effort="1000.0" lower="-0.548" upper="0.548" velocity="0.7" />
+         <limit effort="1000.0" velocity="0.7" lower="-0.548" upper="0.548"/>
          <dynamics damping="0.0" friction="0.5" />
       </joint>
+      <transmission name="${pos}_shoulder_trans">
+         <type>transmission_interface/SimpleTransmission</type>
+         <joint name="${pos}_shoulder">
+               <hardwareInterface>hardware_interface/PositionJointInterface</hardwareInterface>
+         </joint>
+         <actuator name="${pos}_shoulder_actuator">
+               <hardwareInterface>hardware_interface/PositionJointInterface</hardwareInterface>
+               <mechanicalReduction>1</mechanicalReduction>
+         </actuator>
+      </transmission>
    </xacro:macro>
    <xacro:macro name="gen_leg" params="name left">
@@ -124,7 +134,17 @@
          <axis xyz="0 1 0" />
          <origin rpy="0 0 0" xyz="0 ${shift} 0" />
-         <limit effort="1000.0" lower="-2.666" upper="1.548" velocity="0.5" />
+         <limit effort="1000.0" velocity="0.5" lower="-2.666" upper="1.548"/>
          <dynamics damping="0.0" friction="0.0" />
       </joint>
+      <transmission name="${pos}_leg_trans">
+         <type>transmission_interface/SimpleTransmission</type>
+         <joint name="${pos}_leg">
+               <hardwareInterface>hardware_interface/PositionJointInterface</hardwareInterface>
+         </joint>
+         <actuator name="${pos}_leg_actuator">
+               <hardwareInterface>hardware_interface/PositionJointInterface</hardwareInterface>
+               <mechanicalReduction>1</mechanicalReduction>
+         </actuator>
+      </transmission>
       <joint name="${pos}_leg_cover_joint" type="fixed">
          <parent link="${pos}_leg_link" />
@@ -168,7 +188,17 @@
          <axis xyz="0 1 0" />
          <origin rpy="0 0 0" xyz="0.014 0 -${leg_length}" />
-         <limit effort="1000.0" lower="-0.1" upper="2.59" velocity="0.5" />
+         <limit effort="1000.0" velocity="0.5" lower="-2.59" upper="0.1"/>
          <dynamics damping="0.0" friction="0.5" />
       </joint>
+      <transmission name="${pos}_foot_trans">
+         <type>transmission_interface/SimpleTransmission</type>
+         <joint name="${pos}_foot">
+               <hardwareInterface>hardware_interface/PositionJointInterface</hardwareInterface>
+         </joint>
+         <actuator name="${pos}_foot_actuator">
+               <hardwareInterface>hardware_interface/PositionJointInterface</hardwareInterface>
+               <mechanicalReduction>1</mechanicalReduction>
+         </actuator>
+      </transmission>
    </xacro:macro>
    <xacro:macro name="gen_toe" params="name">
