Commit message: update

File: urdf/spotmicroai.urdf (robot description, URDF)
Before this commit: robot SpotMicroAI, 24 links, 23 joints
Links:
- link base_link: geometry collision box size=0.14 0.11 0.07; visual mesh filename=package://spotmicro_description/meshes/spot/stl/mainbody.stl scale=0.001 0.001 0.001
- link front_left_foot_link: geometry collision box size=0.026 0.020 0.115; visual mesh filename=package://spotmicro_description/meshes/spot/stl/lfoot.stl scale=0.001 0.001 0.001
- link front_left_leg_link: geometry collision box size=0.028 0.036 0.12; visual mesh filename=package://spotmicro_description/meshes/spot/stl/larm.stl scale=0.001 0.001 0.001
- link front_left_leg_link_cover: geometry visual mesh filename=package://spotmicro_description/meshes/spot/stl/larm_cover.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 scale=0.001 0.001 0.001
- link front_left_shoulder_link: geometry collision box size=0.044 0.038 0.07; visual mesh filename=package://spotmicro_description/meshes/spot/stl/lshoulder.s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 scale=0.001 0.001 0.001
- link front_left_toe_link: geometry collision sphere radius=0.02; visual mesh filename=package://spotmicro_description/meshes/spot/stl/foot.stl scale=0.001 0.001 0.001
- link front_link: geometry collision box size=0.058 0.11 0.07; visual mesh filename=package://spotmicro_description/meshes/spot/stl/frontpart.s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 scale=0.001 0.001 0.001
- link front_right_foot_link: geometry collision box size=0.026 0.020 0.115; visual mesh filename=package://spotmicro_description/meshes/spot/stl/rfoot.stl scale=0.001 0.001 0.001
- link front_right_leg_link: geometry collision box size=0.028 0.036 0.12; visual mesh filename=package://spotmicro_description/meshes/spot/stl/rarm.stl scale=0.001 0.001 0.001
- link front_right_leg_link_cover: geometry visual mesh filename=package://spotmicro_description/meshes/spot/stl/rarm_cover.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 scale=0.001 0.001 0.001
- link front_right_shoulder_link: geometry collision box size=0.044 0.038 0.07; visual mesh filename=package://spotmicro_description/meshes/spot/stl/rshoulder.s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 scale=0.001 0.001 0.001
- link front_right_toe_link: geometry collision sphere radius=0.02; visual mesh filename=package://spotmicro_description/meshes/spot/stl/foot.stl scale=0.001 0.001 0.001
- link lidar_link: geometry collision box size=0.0985 0.0577 0.07; visual mesh filename=package://spotmicro_description/meshes/spot/stl/rplidar_mai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 scale=0.001 0.001 0.001
- link rear_left_foot_link: geometry collision box size=0.026 0.020 0.115; visual mesh filename=package://spotmicro_description/meshes/spot/stl/lfoot.stl scale=0.001 0.001 0.001
- link rear_left_leg_link: geometry collision box size=0.028 0.036 0.12; visual mesh filename=package://spotmicro_description/meshes/spot/stl/larm.stl scale=0.001 0.001 0.001
- link rear_left_leg_link_cover: geometry visual mesh filename=package://spotmicro_description/meshes/spot/stl/larm_cover.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 scale=0.001 0.001 0.001
- link rear_left_shoulder_link: geometry collision box size=0.044 0.038 0.07; visual mesh filename=package://spotmicro_description/meshes/spot/stl/lshoulder.s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 scale=0.001 0.001 0.001
- link rear_left_toe_link: geometry collision sphere radius=0.02; visual mesh filename=package://spotmicro_description/meshes/spot/stl/foot.stl scale=0.001 0.001 0.001
- link rear_link: geometry collision box size=0.04 0.11 0.07; visual mesh filename=package://spotmicro_description/meshes/spot/stl/backpart.stl scale=0.001 0.001 0.001
- link rear_right_foot_link: geometry collision box size=0.026 0.020 0.115; visual mesh filename=package://spotmicro_description/meshes/spot/stl/rfoot.stl scale=0.001 0.001 0.001
- link rear_right_leg_link: geometry collision box size=0.028 0.036 0.12; visual mesh filename=package://spotmicro_description/meshes/spot/stl/rarm.stl scale=0.001 0.001 0.001
- link rear_right_leg_link_cover: geometry visual mesh filename=package://spotmicro_description/meshes/spot/stl/rarm_cover.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 scale=0.001 0.001 0.001
- link rear_right_shoulder_link: geometry collision box size=0.044 0.038 0.07; visual mesh filename=package://spotmicro_description/meshes/spot/stl/rshoulder.s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 scale=0.001 0.001 0.001
- link rear_right_toe_link: geometry collision sphere radius=0.02; visual mesh filename=package://spotmicro_description/meshes/spot/stl/foot.stl scale=0.001 0.001 0.001

File: urdf/spotmicroai.urdf.xacro (robot description, xacro)
@@ -2,11 +2,11 @@
 <robot xmlns:xacro="http://www.ros.org/wiki/xacro" name="SpotMicroAI">
   <material name="yellow">
-    <color rgba="0.92 0.83 0.0 1"/>
+    <color rgba="0.92 0.83 0.0 1" />
   </material>
   <material name="black">
-    <color rgba="0.1 0.1 0.1 1"/>
+    <color rgba="0.1 0.1 0.1 1" />
   </material>
   <material name="grey">
-    <color rgba="0.6 0.6 0.6 1"/>
+    <color rgba="0.6 0.6 0.6 1" />
   </material>
   <!-- Params -->
@@ -34,25 +34,25 @@
       <visual>
         <xacro:if value="${left}">
-        <geometry>
-          <mesh filename="package://spotmicro_description/meshes/stl/lshoulder.stl" scale="0.001 0.001 0.001"/>
-        </geometry>
-        <origin rpy="0 0 0" xyz="-0.135 -0.02 -0.01"/>
+          <geometry>
+            <mesh filename="package://spotmicro_description/meshes/spot/stl/lshoulder.stl" scale="0.001 0.001 0.001" />
+          </geometry>
+          <origin rpy="0 0 0" xyz="-0.135 -0.02 -0.01" />
         </xacro:if>
         <xacro:unless value="${left}">
-        <geometry>
-          <mesh filename="package://spotmicro_description/meshes/stl/rshoulder.stl" scale="0.001 0.001 0.001"/>
-        </geometry>
-        <origin rpy="0 0 0" xyz="-0.135 -0.09 -0.01"/>
+          <geometry>
+            <mesh filename="package://spotmicro_description/meshes/spot/stl/rshoulder.stl" scale="0.001 0.001 0.001" />
+          </geometry>
+          <origin rpy="0 0 0" xyz="-0.135 -0.09 -0.01" />
         </xacro:unless>
-        <material name="black"/>
+        <material name="black" />
       </visual>
       <collision>
         <geometry>
-          <box size="${shoulder_length} ${shoulder_width} ${body_height}"/>
-        </geometry>
-        <origin rpy="0 0 0" xyz="0 0 0"/>
+          <box size="${shoulder_length} ${shoulder_width} ${body_height}" />
+        </geometry>
+        <origin rpy="0 0 0" xyz="0 0 0" />
       </collision>
       <inertial>
-        <mass value="0.10"/>
+        <mass value="0.10" />
         <inertia ixx="100" ixy="0" ixz="0" iyy="100" iyz="0" izz="100" />
       </inertial>
@@ -61,10 +61,10 @@
   <xacro:macro name="gen_shoulder_joint" params="pos shiftx shifty">
     <joint name="${pos}_shoulder" type="revolute">
-      <parent link="base_link"/>
-      <child link="${pos}_shoulder_link"/>
-      <axis xyz="1 0 0"/>
-      <origin rpy="0 0 0" xyz="${shiftx} ${shifty} 0"/>
-      <limit effort="1000.0" lower="-0.548" upper="0.548" velocity="0.7"/>
-      <dynamics damping="0.0" friction="0.5"/>
+      <parent link="base_link" />
+      <child link="${pos}_shoulder_link" />
+      <axis xyz="1 0 0" />
+      <origin rpy="0 0 0" xyz="${shiftx} ${shifty} 0" />
+      <limit effort="1000.0" lower="-0.548" upper="0.548" velocity="0.7" />
+      <dynamics damping="0.0" friction="0.5" />
     </joint>
   </xacro:macro>
@@ -73,16 +73,16 @@
       <visual>
         <xacro:if value="${left}">
-        <geometry>
-          <mesh filename="package://spotmicro_description/meshes/stl/larm_cover.stl" scale="0.001 0.001 0.001"/>
-        </geometry>
-        <origin rpy="0 0 0" xyz="-0.125 0.04 -0.02"/>
+          <geometry>
+            <mesh filename="package://spotmicro_description/meshes/spot/stl/larm_cover.stl" scale="0.001 0.001 0.001" />
+          </geometry>
+          <origin rpy="0 0 0" xyz="-0.125 0.04 -0.02" />
         </xacro:if>
         <xacro:unless value="${left}">
-        <geometry>
-          <mesh filename="package://spotmicro_description/meshes/stl/rarm_cover.stl" scale="0.001 0.001 0.001"/>
-        </geometry>
-        <origin rpy="0 0 0" xyz="-0.125 -0.15 -0.02"/>
+          <geometry>
+            <mesh filename="package://spotmicro_description/meshes/spot/stl/rarm_cover.stl" scale="0.001 0.001 0.001" />
+          </geometry>
+          <origin rpy="0 0 0" xyz="-0.125 -0.15 -0.02" />
         </xacro:unless>
-        <material name="yellow"/>
+        <material name="yellow" />
       </visual>
     </link>
@@ -90,17 +90,17 @@
       <visual>
         <xacro:if value="${left}">
-        <geometry>
-          <mesh filename="package://spotmicro_description/meshes/stl/larm.stl" scale="0.001 0.001 0.001"/>
-        </geometry>
-        <origin rpy="0 0 0" xyz="-0.125 0.04 -0.02"/>
+          <geometry>
+            <mesh filename="package://spotmicro_description/meshes/spot/stl/larm.stl" scale="0.001 0.001 0.001" />
+          </geometry>
+          <origin rpy="0 0 0" xyz="-0.125 0.04 -0.02" />
         </xacro:if>
         <xacro:unless value="${left}">
-        <geometry>
-          <mesh filename="package://spotmicro_description/meshes/stl/rarm.stl" scale="0.001 0.001 0.001"/>
-        </geometry>
-        <origin rpy="0 0 0" xyz="-0.125 -0.15 -0.02"/>
+          <geometry>
+            <mesh filename="package://spotmicro_description/meshes/spot/stl/rarm.stl" scale="0.001 0.001 0.001" />
+          </geometry>
+          <origin rpy="0 0 0" xyz="-0.125 -0.15 -0.02" />
         </xacro:unless>
-        <material name="black"/>
-<!--        <geometry>
+        <material name="black" />
+        <!--        <geometry>
           <box size="0.028 0.036 ${leg_length}"/>
         </geometry>
@@ -109,11 +109,11 @@
       </visual>
       <collision>
-        <origin rpy="0.0 0.0 0.0" xyz="0.0 0.0 -0.050"/>
-        <geometry>
-          <box size="0.028 0.036 ${leg_length}"/>
+        <origin rpy="0.0 0.0 0.0" xyz="0.0 0.0 -0.050" />
+        <geometry>
+          <box size="0.028 0.036 ${leg_length}" />
         </geometry>
       </collision>
       <inertial>
-        <mass value="0.15"/>
+        <mass value="0.15" />
         <inertia ixx="1000" ixy="0" ixz="0" iyy="1000" iyz="0" izz="1000" />
       </inertial>
@@ -122,16 +122,16 @@
   <xacro:macro name="gen_leg_joint" params="pos shift">
     <joint name="${pos}_leg" type="revolute">
-      <parent link="${pos}_shoulder_link"/>
-      <child link="${pos}_leg_link"/>
-      <axis xyz="0 1 0"/>
-      <origin rpy="0 0 0" xyz="0 ${shift} 0"/>
-      <limit effort="1000.0" lower="-2.666" upper="1.548" velocity="0.5"/>
-      <dynamics damping="0.0" friction="0.0"/>
+      <parent link="${pos}_shoulder_link" />
+      <child link="${pos}_leg_link" />
+      <axis xyz="0 1 0" />
+      <origin rpy="0 0 0" xyz="0 ${shift} 0" />
+      <limit effort="1000.0" lower="-2.666" upper="1.548" velocity="0.5" />
+      <dynamics damping="0.0" friction="0.0" />
     </joint>
     <joint name="${pos}_leg_cover_joint" type="fixed">
-    <parent link="${pos}_leg_link"/>
-    <child link="${pos}_leg_link_cover"/>
-        <origin xyz="0 0 0"/>
-  </joint>
+      <parent link="${pos}_leg_link" />
+      <child link="${pos}_leg_link_cover" />
+      <origin xyz="0 0 0" />
+    </joint>
   </xacro:macro>
   <xacro:macro name="gen_foot" params="name left">
@@ -139,25 +139,25 @@
       <visual>
         <xacro:if value="${left}">
-        <geometry>
-          <mesh filename="package://spotmicro_description/meshes/stl/lfoot.stl" scale="0.001 0.001 0.001"/>
-        </geometry>
-        <origin rpy="0 0 0" xyz="-0.120 0.04 0.1"/>
+          <geometry>
+            <mesh filename="package://spotmicro_description/meshes/spot/stl/lfoot.stl" scale="0.001 0.001 0.001" />
+          </geometry>
+          <origin rpy="0 0 0" xyz="-0.120 0.04 0.1" />
         </xacro:if>
         <xacro:unless value="${left}">
-        <geometry>
-          <mesh filename="package://spotmicro_description/meshes/stl/rfoot.stl" scale="0.001 0.001 0.001"/>
-        </geometry>
-        <origin rpy="0 0 0" xyz="-0.120 -0.15 0.1"/>
+          <geometry>
+            <mesh filename="package://spotmicro_description/meshes/spot/stl/rfoot.stl" scale="0.001 0.001 0.001" />
+          </geometry>
+          <origin rpy="0 0 0" xyz="-0.120 -0.15 0.1" />
         </xacro:unless>
-        <material name="black"/>
+        <material name="black" />
       </visual>
       <collision>
         <geometry>
-          <box size="0.026 0.020 ${foot_length}"/>
-        </geometry>
-        <origin rpy="0.0 0.0 0.0" xyz="0.0 0.0 -0.050"/>
+          <box size="0.026 0.020 ${foot_length}" />
+        </geometry>
+        <origin rpy="0.0 0.0 0.0" xyz="0.0 0.0 -0.050" />
       </collision>
       <inertial>
-        <mass value="0.1"/>
+        <mass value="0.1" />
         <inertia ixx="1000" ixy="0" ixz="0" iyy="1000" iyz="0" izz="1000" />
       </inertial>
@@ -166,10 +166,10 @@
   <xacro:macro name="gen_foot_joint" params="pos">
     <joint name="${pos}_foot" type="revolute">
-      <parent link="${pos}_leg_link"/>
-      <child link="${pos}_foot_link"/>
-      <axis xyz="0 1 0"/>
-      <origin rpy="0 0 0" xyz="-0.01 0 -${leg_length}"/>
-      <limit effort="1000.0" lower="-0.1" upper="2.59" velocity="0.5"/>
-      <dynamics damping="0.0" friction="0.5"/>
+      <parent link="${pos}_leg_link" />
+      <child link="${pos}_foot_link" />
+      <axis xyz="0 1 0" />
+      <origin rpy="0 0 0" xyz="-0.01 0 -${leg_length}" />
+      <limit effort="1000.0" lower="-0.1" upper="2.59" velocity="0.5" />
+      <dynamics damping="0.0" friction="0.5" />
     </joint>
   </xacro:macro>
@@ -178,8 +178,8 @@
       <visual>
         <geometry>
-        <mesh filename="package://spotmicro_description/meshes/stl/foot.stl" scale="0.001 0.001 0.001"/>
-        </geometry>
-        <origin rpy="0 -0.40010 0" xyz="0 -0.01 0"/>
-        <material name="grey"/>
+          <mesh filename="package://spotmicro_description/meshes/spot/stl/foot.stl" scale="0.001 0.001 0.001" />
+        </geometry>
+        <origin rpy="0 -0.40010 0" xyz="0 -0.01 0" />
+        <material name="grey" />
       </visual>
       <collision>
@@ -187,29 +187,29 @@
           <sphere radius="${toe_radius}" />
         </geometry>
-        <origin rpy="0 0 0" xyz="0 0 0"/>
+        <origin rpy="0 0 0" xyz="0 0 0" />
         <contact_coefficients mu="1.1" />
       </collision>
       <inertial>
-        <mass value="0.05"/>
+        <mass value="0.05" />
         <inertia ixx="1000" ixy="0" ixz="0" iyy="1000" iyz="0" izz="1000" />
       </inertial>
     </link>
   </xacro:macro>
- <xacro:macro name="gen_toe_joint" params="pos">
+  <xacro:macro name="gen_toe_joint" params="pos">
     <joint name="${pos}_toe" type="fixed">
-      <parent link="${pos}_foot_link"/>
-      <child link="${pos}_toe_link"/>
-      <origin xyz="0 0 -${foot_length}"/>
+      <parent link="${pos}_foot_link" />
+      <child link="${pos}_toe_link" />
+      <origin xyz="0 0 -${foot_length}" />
     </joint>
   </xacro:macro>
   <xacro:macro name="gen_full_leg_joint" params="pos shiftx shifty shift left">
-    <xacro:gen_shoulder name="${pos}_shoulder_link" left="${left}"/>
-    <xacro:gen_leg name="${pos}_leg_link" left="${left}"/>
-    <xacro:gen_foot name="${pos}_foot_link" left="${left}"/>
-    <xacro:gen_toe name="${pos}_toe_link"/>
-    <xacro:gen_shoulder_joint pos="${pos}" shiftx="${shiftx}" shifty="${shifty}"/>
-    <xacro:gen_leg_joint pos="${pos}" shift="${shift}"/>
-    <xacro:gen_foot_joint pos="${pos}"/>
-    <xacro:gen_toe_joint pos="${pos}"/>
+    <xacro:gen_shoulder name="${pos}_shoulder_link" left="${left}" />
+    <xacro:gen_leg name="${pos}_leg_link" left="${left}" />
+    <xacro:gen_foot name="${pos}_foot_link" left="${left}" />
+    <xacro:gen_toe name="${pos}_toe_link" />
+    <xacro:gen_shoulder_joint pos="${pos}" shiftx="${shiftx}" shifty="${shifty}" />
+    <xacro:gen_leg_joint pos="${pos}" shift="${shift}" />
+    <xacro:gen_foot_joint pos="${pos}" />
+    <xacro:gen_toe_joint pos="${pos}" />
   </xacro:macro>
   <!-- Robot Body -->
@@ -217,95 +217,95 @@
     <visual>
       <geometry>
-        <mesh filename="package://spotmicro_description/meshes/stl/mainbody.stl" scale="0.001 0.001 0.001"/>
-      </geometry>
-      <material name="black"/>
-      <origin rpy="0 0 0" xyz="-0.045 -0.060 -0.015"/>
+        <mesh filename="package://spotmicro_description/meshes/spot/stl/mainbody.stl" scale="0.001 0.001 0.001" />
+      </geometry>
+      <material name="black" />
+      <origin rpy="0 0 0" xyz="-0.045 -0.060 -0.015" />
     </visual>
     <collision>
       <geometry>
-        <box size="${body_length} ${body_width} ${body_height}"/>
-      </geometry>
-      <origin rpy="0 0 0" xyz="0 0 0"/>
+        <box size="${body_length} ${body_width} ${body_height}" />
+      </geometry>
+      <origin rpy="0 0 0" xyz="0 0 0" />
     </collision>
     <inertial>
-      <mass value="2.80"/>
+      <mass value="2.80" />
       <inertia ixx="100" ixy="0" ixz="0" iyy="100" iyz="0" izz="100" />
     </inertial>
   </link>
   <!-- Lidar Backpack -->
-   <link name="lidar_link">
+  <link name="lidar_link">
     <visual>
       <geometry>
-        <mesh filename="package://spotmicro_description/meshes/stl/rplidar_main.STL" scale="0.001 0.001 0.001"/>
-      </geometry>
-      <material name="black"/>
-      <origin rpy="1.57075 0 0" xyz="${-lidar_length/2-0.015} ${lidar_width/2} 0"/>
+        <mesh filename="package://spotmicro_description/meshes/spot/stl/rplidar_main.STL" scale="0.001 0.001 0.001" />
+      </geometry>
+      <material name="black" />
+      <origin rpy="1.57075 0 0" xyz="${-lidar_length/2-0.015} ${lidar_width/2} 0" />
     </visual>
     <collision>
       <geometry>
-        <box size="${lidar_length} ${lidar_width} ${lidar_height}"/>
-      </geometry>
-      <origin rpy="0 0 0" xyz="0 0 0"/>
+        <box size="${lidar_length} ${lidar_width} ${lidar_height}" />
+      </geometry>
+      <origin rpy="0 0 0" xyz="0 0 0" />
     </collision>
     <inertial>
-      <mass value="0.50"/>
+      <mass value="0.50" />
       <inertia ixx="100" ixy="0" ixz="0" iyy="100" iyz="0" izz="100" />
     </inertial>
   </link>
   <joint name="base_lidar" type="fixed">
-    <parent link="base_link"/>
-    <child link="lidar_link"/>
-        <origin xyz="0 0 ${body_height/2}"/>
+    <parent link="base_link" />
+    <child link="lidar_link" />
+    <origin xyz="0 0 ${body_height/2}" />
   </joint>
   <link name="rear_link">
     <visual>
       <geometry>
-        <mesh filename="package://spotmicro_description/meshes/stl/backpart.stl" scale="0.001 0.001 0.001"/>
-      </geometry>
-      <origin rpy="0 0 0" xyz="-0.040 -0.060 -0.0140"/>
-      <material name="yellow"/>
+        <mesh filename="package://spotmicro_description/meshes/spot/stl/backpart.stl" scale="0.001 0.001 0.001" />
+      </geometry>
+      <origin rpy="0 0 0" xyz="-0.040 -0.060 -0.0140" />
+      <material name="yellow" />
     </visual>
     <collision>
       <geometry>
-        <box size="${rear_length} ${body_width} ${body_height}"/>
-      </geometry>
-      <origin rpy="0 0 0" xyz="0.135 0 0"/>
+        <box size="${rear_length} ${body_width} ${body_height}" />
+      </geometry>
+      <origin rpy="0 0 0" xyz="0.135 0 0" />
     </collision>
     <inertial>
-      <mass value="0.20"/>
+      <mass value="0.20" />
       <inertia ixx="100" ixy="0" ixz="0" iyy="100" iyz="0" izz="100" />
     </inertial>
   </link>
   <joint name="base_rear" type="fixed">
-    <parent link="base_link"/>
-    <child link="rear_link"/>
+    <parent link="base_link" />
+    <child link="rear_link" />
   </joint>
   <link name="front_link">
     <visual>
       <geometry>
-        <mesh filename="package://spotmicro_description/meshes/stl/frontpart.stl" scale="0.001 0.001 0.001"/>
-      </geometry>
-      <origin rpy="0 0 0" xyz="-0.040 -0.060 -0.0140"/>
-      <material name="yellow"/>
+        <mesh filename="package://spotmicro_description/meshes/spot/stl/frontpart.stl" scale="0.001 0.001 0.001" />
+      </geometry>
+      <origin rpy="0 0 0" xyz="-0.040 -0.060 -0.0140" />
+      <material name="yellow" />
     </visual>
     <collision>
       <geometry>
-        <box size="${front_length} ${body_width} ${body_height}"/>
-      </geometry>
-      <origin rpy="0 0 0" xyz="-0.145 0 0"/>
+        <box size="${front_length} ${body_width} ${body_height}" />
+      </geometry>
+      <origin rpy="0 0 0" xyz="-0.145 0 0" />
     </collision>
     <inertial>
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