Commit message: update

File: urdf/hyq.urdf (robot description, URDF)
Before this commit: robot hyq, 19 links, 18 joints
Links:
- removed link hokuyo_link
- removed link lf_foot
- removed link lf_hipassembly
- removed link lf_lowerleg
- removed link lf_upperleg
- removed link lh_foot
- removed link lh_hipassembly
- removed link lh_lowerleg
- removed link lh_upperleg
- removed link rf_foot
- removed link rf_hipassembly
- removed link rf_lowerleg
- removed link rf_upperleg
- removed link rh_foot
- removed link rh_hipassembly
- removed link rh_lowerleg
- removed link rh_upperleg
- added link hokuyo_frame, mass 1e-5; collision box size=0.1 0.1 0.1; visual mesh filename=package://spotmicro_description/meshes/hyq/hokuyo.dae scale=1 1 1
- added link l_front_hipassembly_link, mass 2.93; collision mesh filename=package://spotmicro_description/meshes/hyq/leg/hipassembly.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 scale=1 1 1; visual mesh filename=package://spotmicro_description/meshes/hyq/leg/hipassembly.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 scale=1 1 1
- added link l_front_lower_leg_link, mass 0.881; collision mesh filename=package://spotmicro_description/meshes/hyq/leg/lowerleg.dae scale=1 1 1; visual mesh filename=package://spotmicro_description/meshes/hyq/leg/lowerleg.dae scale=1 1 1
- added link l_front_toe_link, mass 0.1; collision sphere radius=0.02175; visual sphere radius=0.02175
- added link l_front_upper_leg_link, mass 2.638; collision mesh filename=package://spotmicro_description/meshes/hyq/leg/upperleg.dae scale=1 1 1; visual mesh filename=package://spotmicro_description/meshes/hyq/leg/upperleg.dae scale=1 1 1
- added link l_rear_hipassembly_link, mass 2.93; collision mesh filename=package://spotmicro_description/meshes/hyq/leg/hipassembly.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 scale=1 1 1; visual mesh filename=package://spotmicro_description/meshes/hyq/leg/hipassembly.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 scale=1 1 1
- added link l_rear_lower_leg_link, mass 0.881; collision mesh filename=package://spotmicro_description/meshes/hyq/leg/lowerleg.dae scale=1 1 1; visual mesh filename=package://spotmicro_description/meshes/hyq/leg/lowerleg.dae scale=1 1 1
- added link l_rear_toe_link, mass 0.1; collision sphere radius=0.02175; visual sphere radius=0.02175
- added link l_rear_upper_leg_link, mass 2.638; collision mesh filename=package://spotmicro_description/meshes/hyq/leg/upperleg.dae scale=1 1 1; visual mesh filename=package://spotmicro_description/meshes/hyq/leg/upperleg.dae scale=1 1 1
- added link r_front_hipassembly_link, mass 2.93; collision mesh filename=package://spotmicro_description/meshes/hyq/leg/hipassembly.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 scale=1 1 1; visual mesh filename=package://spotmicro_description/meshes/hyq/leg/hipassembly.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 scale=1 1 1
- added link r_front_lower_leg_link, mass 0.881; collision mesh filename=package://spotmicro_description/meshes/hyq/leg/lowerleg.dae scale=1 1 1; visual mesh filename=package://spotmicro_description/meshes/hyq/leg/lowerleg.dae scale=1 1 1
- added link r_front_toe_link, mass 0.1; collision sphere radius=0.02175; visual sphere radius=0.02175
- added link r_front_upper_leg_link, mass 2.638; collision mesh filename=package://spotmicro_description/meshes/hyq/leg/upperleg.dae scale=1 1 1; visual mesh filename=package://spotmicro_description/meshes/hyq/leg/upperleg.dae scale=1 1 1
- added link r_rear_hipassembly_link, mass 2.93; collision mesh filename=package://spotmicro_description/meshes/hyq/leg/hipassembly.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 scale=1 1 1; visual mesh filename=package://spotmicro_description/meshes/hyq/leg/hipassembly.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 scale=1 1 1
- added link r_rear_lower_leg_link, mass 0.881; collision mesh filename=package://spotmicro_description/meshes/hyq/leg/lowerleg.dae scale=1 1 1; visual mesh filename=package://spotmicro_description/meshes/hyq/leg/lowerleg.dae scale=1 1 1
- added link r_rear_toe_link, mass 0.1; collision sphere radius=0.02175; visual sphere radius=0.02175
- added link r_rear_upper_leg_link, mass 2.638; collision mesh filename=package://spotmicro_description/meshes/hyq/leg/upperleg.dae scale=1 1 1; visual mesh filename=package://spotmicro_description/meshes/hyq/leg/upperleg.dae scale=1 1 1
Joints:
- removed joint lf_foot_joint
- removed joint lf_haa_joint
- removed joint lf_hfe_joint
- removed joint lf_kfe_joint
- removed joint lh_foot_joint
- removed joint lh_haa_joint
- removed joint lh_hfe_joint
- removed joint lh_kfe_joint
- removed joint rf_foot_joint
- removed joint rf_haa_joint
- removed joint rf_hfe_joint
- removed joint rf_kfe_joint
- removed joint rh_foot_joint
- removed joint rh_haa_joint
- removed joint rh_hfe_joint
- removed joint rh_kfe_joint
- added joint l_front_hipassembly_joint: type revolute, parent trunk, child l_front_hipassembly_link, origin xyz=0.3735 0.207 0 rpy=0 1.57079632679 3.14159265359, axis 0 0 1, limit lower=-1.2217304764 upper=0.436332312999 effort=150 velocity=12.0
- added joint l_front_lower_leg_joint: type revolute, parent l_front_upper_leg_link, child l_front_lower_leg_link, origin xyz=0.35 0 0 rpy=0 0 0, axis 0 0 1, limit lower=-2.44346095279 upper=-0.349065850399 effort=150 velocity=12.0
- added joint l_front_toe_joint: type fixed, parent l_front_lower_leg_link, child l_front_toe_link, origin xyz=0.346 0 0 rpy=1.57079632679 0 -1.57079632679
- added joint l_front_upper_leg_joint: type revolute, parent l_front_hipassembly_link, child l_front_upper_leg_link, origin xyz=0.08 0 0 rpy=1.57079632679 0 0, axis 0 0 1, limit lower=-0.872664625997 upper=1.2217304764 effort=150 velocity=12.0
- added joint l_rear_hipasembly_joint: type revolute, parent trunk, child l_rear_hipassembly_link, origin xyz=-0.3735 0.207 0 rpy=0 1.57079632679 3.14159265359, axis 0 0 1, limit lower=-1.2217304764 upper=0.436332312999 effort=150 velocity=12.0
- added joint l_rear_lower_leg_joint: type revolute, parent l_rear_upper_leg_link, child l_rear_lower_leg_link, origin xyz=0.35 0 0 rpy=0 0 0, axis 0 0 1, limit lower=0.349065850399 upper=2.44346095279 effort=150 velocity=12.0
- added joint l_rear_toe_joint: type fixed, parent l_rear_lower_leg_link, child l_rear_toe_link, origin xyz=0.346 0 0 rpy=1.57079632679 0 -1.57079632679
- added joint l_rear_upper_leg_joint: type revolute, parent l_rear_hipassembly_link, child l_rear_upper_leg_link, origin xyz=0.08 0 0 rpy=1.57079632679 0 0, axis 0 0 1, limit lower=-1.2217304764 upper=0.872664625997 effort=150 velocity=12.0
- added joint r_front_hipassembly_joint: type revolute, parent trunk, child r_front_hipassembly_link, origin xyz=0.3735 -0.207 0 rpy=0 1.57079632679 0, axis 0 0 1, limit lower=-1.2217304764 upper=0.436332312999 effort=150 velocity=12.0
- added joint r_front_lower_leg_joint: type revolute, parent r_front_upper_leg_link, child r_front_lower_leg_link, origin xyz=0.35 0 0 rpy=0 0 0, axis 0 0 1, limit lower=-2.44346095279 upper=-0.349065850399 effort=150 velocity=12.0
- added joint r_front_toe_joint: type fixed, parent r_front_lower_leg_link, child r_front_toe_link, origin xyz=0.346 0 0 rpy=1.57079632679 0 -1.57079632679
- added joint r_front_upper_leg_joint: type revolute, parent r_front_hipassembly_link, child r_front_upper_leg_link, origin xyz=0.08 0 0 rpy=-1.57079632679 0 0, axis 0 0 1, limit lower=-0.872664625997 upper=1.2217304764 effort=150 velocity=12.0
- added joint r_rear_hipassembly_joint: type revolute, parent trunk, child r_rear_hipassembly_link, origin xyz=-0.3735 -0.207 0 rpy=0 1.57079632679 0, axis 0 0 1, limit lower=-1.2217304764 upper=0.436332312999 effort=150 velocity=12.0
- added joint r_rear_lower_leg_joint: type revolute, parent r_rear_upper_leg_link, child r_rear_lower_leg_link, origin xyz=0.35 0 0 rpy=0 0 0, axis 0 0 1, limit lower=0.349065850399 upper=2.44346095279 effort=150 velocity=12.0
- added joint r_rear_toe_joint: type fixed, parent r_rear_lower_leg_link, child r_rear_toe_link, origin xyz=0.346 0 0 rpy=1.57079632679 0 -1.57079632679
- added joint r_rear_upper_leg_joint: type revolute, parent r_rear_hipassembly_link, child r_rear_upper_leg_link, origin xyz=0.08 0 0 rpy=-1.57079632679 0 0, axis 0 0 1, limit lower=-1.2217304764 upper=0.872664625997 effort=150 velocity=12.0
- joint hokuyo_joint: child hokuyo_link -> hokuyo_frame

File: urdf/spotmicroai.urdf (robot description, URDF)
Before this commit: robot SpotMicroAI, 24 links, 23 joints
Links:
- removed link lidar_link
- added link base_inertia, mass 2.80; collision box size=0.14 0.11 0.07; visual mesh filename=package://spotmicro_description/meshes/spot/stl/mainbody.stl scale=0.001 0.001 0.001
- added link lidar_frame, mass 0.50; collision box size=0.0985 0.0577 0.07; visual mesh filename=package://spotmicro_description/meshes/spot/rplidar_main.STL scale=0.001 0.001 0.001
- link base_link: mass 2.80 -> None; geometry 
- link front_left_foot_link: geometry collision box size=0.026 0.020 0.13; visual mesh filename=package://spotmicro_description/meshes/spot/stl/lfoot.stl scale=0.001 0.001 0.001
- link front_left_leg_link: geometry collision box size=0.028 0.036 0.109; visual mesh filename=package://spotmicro_description/meshes/spot/stl/larm.stl scale=0.001 0.001 0.001
- link front_right_foot_link: geometry collision box size=0.026 0.020 0.13; visual mesh filename=package://spotmicro_description/meshes/spot/stl/rfoot.stl scale=0.001 0.001 0.001
- link front_right_leg_link: geometry collision box size=0.028 0.036 0.109; visual mesh filename=package://spotmicro_description/meshes/spot/stl/rarm.stl scale=0.001 0.001 0.001
- link rear_left_foot_link: geometry collision box size=0.026 0.020 0.13; visual mesh filename=package://spotmicro_description/meshes/spot/stl/lfoot.stl scale=0.001 0.001 0.001
- link rear_left_leg_link: geometry collision box size=0.028 0.036 0.109; visual mesh filename=package://spotmicro_description/meshes/spot/stl/larm.stl scale=0.001 0.001 0.001
- link rear_right_foot_link: geometry collision box size=0.026 0.020 0.13; visual mesh filename=package://spotmicro_description/meshes/spot/stl/rfoot.stl scale=0.001 0.001 0.001
- link rear_right_leg_link: geometry collision box size=0.028 0.036 0.109; visual mesh filename=package://spotmicro_description/meshes/spot/stl/rarm.stl scale=0.001 0.001 0.001
Joints:
- added joint base_inertia_joint: type fixed, parent base_link, child base_inertia
- joint base_lidar: child lidar_link -> lidar_frame
- joint front_left_foot: limit lower=-0.1 upper=2.59 effort=1000.0 velocity=0.5 -> lower=-2.59 upper=0.1 effort=1000.0 velocity=0.5; origin xyz=-0.01 0 -0.12 rpy=0 0 0 -> xyz=0.014 0 -0.109 rpy=0 0 0
- joint front_left_leg: origin xyz=0 -0.052 0 rpy=0 0 0 -> xyz=0 0.055 0 rpy=0 0 0
- joint front_left_shoulder: origin xyz=-0.093 -0.036 0 rpy=0 0 0 -> xyz=0.093 0.0395 0 rpy=0 0 0
- joint front_left_toe: origin xyz=0 0 -0.115 -> xyz=0 0 -0.13
- joint front_right_foot: limit lower=-0.1 upper=2.59 effort=1000.0 velocity=0.5 -> lower=-2.59 upper=0.1 effort=1000.0 velocity=0.5; origin xyz=-0.01 0 -0.12 rpy=0 0 0 -> xyz=0.014 0 -0.109 rpy=0 0 0
- joint front_right_leg: origin xyz=0 0.052 0 rpy=0 0 0 -> xyz=0 -0.055 0 rpy=0 0 0
- joint front_right_shoulder: origin xyz=-0.093 0.036 0 rpy=0 0 0 -> xyz=0.093 -0.0395 0 rpy=0 0 0
- joint front_right_toe: origin xyz=0 0 -0.115 -> xyz=0 0 -0.13
- joint rear_left_foot: limit lower=-0.1 upper=2.59 effort=1000.0 velocity=0.5 -> lower=-2.59 upper=0.1 effort=1000.0 velocity=0.5; origin xyz=-0.01 0 -0.12 rpy=0 0 0 -> xyz=0.014 0 -0.109 rpy=0 0 0
- joint rear_left_leg: origin xyz=0 -0.052 0 rpy=0 0 0 -> xyz=0 0.055 0 rpy=0 0 0
- joint rear_left_shoulder: origin xyz=0.093 -0.036 0 rpy=0 0 0 -> xyz=-0.093 0.0395 0 rpy=0 0 0
- joint rear_left_toe: origin xyz=0 0 -0.115 -> xyz=0 0 -0.13
- joint rear_right_foot: limit lower=-0.1 upper=2.59 effort=1000.0 velocity=0.5 -> lower=-2.59 upper=0.1 effort=1000.0 velocity=0.5; origin xyz=-0.01 0 -0.12 rpy=0 0 0 -> xyz=0.014 0 -0.109 rpy=0 0 0
- joint rear_right_leg: origin xyz=0 0.052 0 rpy=0 0 0 -> xyz=0 -0.055 0 rpy=0 0 0
- joint rear_right_shoulder: origin xyz=0.093 0.036 0 rpy=0 0 0 -> xyz=-0.093 -0.0395 0 rpy=0 0 0
- joint rear_right_toe: origin xyz=0 0 -0.115 -> xyz=0 0 -0.13
